File: main_board/hot_table.kicad_sch (KiCad schematic)
At the start: 57 parts, among them J1 HV_CONN, J2 FUN_12V_CONN, J3 T_CONTROL_CONN, J4 USB_B_Mini, J5 SWD_CONN, J6 HMI_CONN, J7 PSU_12V_CONN, J8 BUZZER_CONN, K1 FINDER-36.11, K2 FINDER-36.11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

Commit message: Change comment
Other:
- note added: "PF0 (FT) - OSC_IN PF1 (FT) - OSC_OUT PA0 - USART2_CTS, RTC_TAMP2, WKUP1, ADC_IN0 PA1 - USART2_RTS, ADC_IN1 PA2 - USART2_TX, ADC_IN2, WKUP4 PA3 - USART2_RX, ADC_IN3 PA4 - SPI1_NSS, TIM14_CH1, USART2_CK, ADC_IN4 PA5 - SPI1_SCK, ADC_IN5 PA6 - SPI1_MISO, TIM3_CH1, TIM1_BKIN, TIM16_CH1, ADC_IN6 PA7 - SPI1_MOSI, TIM3_CH2, TIM14_CH1, TIM1_CH1N, TIM17_CH1, ADC_IN7 PA9 (FT) - USART1_TX, TIM1_CH2, TIM15_BK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"
- note removed: "PF0 (FT) - OSC_IN PF1 (FT) - OSC_OUT PA0 - USART2_CTS, USART4_TX, RTC_TAMP2, WKUP1, ADC_IN0 PA1 - USART2_RTS, TIM15_CH1N, USART4_RX, ADC_IN1 PA2 - USART2_TX, TIM15_CH1, ADC_IN2, WKUP4 PA3 - USART2_RX, TIM15_CH2, ADC_IN3 PA4 - SPI1_NSS, TIM14_CH1, USART2_CK, ADC_IN4 PA5 - SPI1_SCK, ADC_IN5 PA6 - SPI1_MISO, TIM3_CH1, TIM1_BKIN, TIM16_CH1, USART3_CTS, ADC_IN6 PA7 - SPI1_MOSI, TIM3_CH2, TIM14_CH1, TI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"
Changed lines of the file:
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@@
     (effects (font (size 1.27 1.27)) (justify left bottom))
   )
-  (text "PF0 (FT) - OSC_IN\nPF1 (FT) - OSC_OUT\n\nPA0 - USART2_CTS, USART4_TX, RTC_TAMP2, WKUP1, ADC_IN0\nPA1 - USART2_RTS, TIM15_CH1N, USART4_RX, ADC_IN1\nPA2 - USART2_TX, TIM15_CH1, ADC_IN2, WKUP4\nPA3 - USART2_RX, TIM15_CH2, ADC_IN3\nPA4 - SPI1_NSS, TIM14_CH1, USART2_CK, ADC_IN4\nPA5 - SPI1_SCK, ADC_IN5\nPA6 - SPI1_MISO, TIM3_CH1, TIM1_BKIN, TIM16_CH1, USART3_CTS, ADC_IN6\nPA7 - SPI1_MOSI, TIM3_CH2, TIM14_CH1, TIM1_CH1N, TIM17_CH1, ADC_IN7\nPA9 (FT) - USART1_TX, TIM1_CH2, TIM15_BKIN, I2C1_SCK\nPA10 (FT) - USART1_RX, TIM1_CH3, TIM17_BKIN, I2C1_SDA\nPA11 (FT) - USART1_CTS, TIM1_CH4, USB_DM\nPA12 (FT) - USART1_RTS, TIM1_ETR, USB_DP\nPA13 (FT) - SWDIO\nPA14 (FT) - SWCLK\n\nPB1 - TIM3_CH4, USART3_RTS, TIM14_CH1, TIM1_CH3N, ADC_IN9"
+  (text "PF0 (FT) - OSC_IN\nPF1 (FT) - OSC_OUT\n\nPA0 - USART2_CTS, RTC_TAMP2, WKUP1, ADC_IN0\nPA1 - USART2_RTS, ADC_IN1\nPA2 - USART2_TX, ADC_IN2, WKUP4\nPA3 - USART2_RX, ADC_IN3\nPA4 - SPI1_NSS, TIM14_CH1, USART2_CK, ADC_IN4\nPA5 - SPI1_SCK, ADC_IN5\nPA6 - SPI1_MISO, TIM3_CH1, TIM1_BKIN, TIM16_CH1, ADC_IN6\nPA7 - SPI1_MOSI, TIM3_CH2, TIM14_CH1, TIM1_CH1N, TIM17_CH1, ADC_IN7\nPA9 (FT) - USART1_TX, TIM1_CH2, TIM15_BKIN, I2C1_SCK\nPA10 (FT) - USART1_RX, TIM1_CH3, TIM17_BKIN, I2C1_SDA\nPA11 (FT) - USART1_CTS, TIM1_CH4, USB_DM\nPA12 (FT) - USART1_RTS, TIM1_ETR, USB_DP\nPA13 (FT) - SWDIO\nPA14 (FT) - SWCLK\n\nPB1 - TIM3_CH4, USART3_RTS, TIM14_CH1, TIM1_CH3N, ADC_IN9"
     (at 201.93 125.73 0)
     (effects (font (size 1.27 1.27)) (justify left bottom))
